File: Final_project_rbree/Final_project_rbree.kicad_sch (KiCad schematic)
At the start: 48 parts, among them J1 Conn_01x02_Pin, J2 Conn_01x02_Pin, Q1 MMBT3904, Q2 AO3401A, U1 TL431, U2 LTV-817, U3 B1212, U4 2N7002, U7 NE555

Commit message: Post-interview build
Slightly rewired PCB, schematics still have changes to be made.
Parts:
- H1, H2, H3, H4: footprint MountingHole:MountingHole_3mm -> MountingHole:MountingHole_3.2mm_M3
Changed lines of the file:
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@@
 			)
 		)
-		(property "Footprint" "MountingHole:MountingHole_3mm"
+		(property "Footprint" "MountingHole:MountingHole_3.2mm_M3"
 			(at 331.47 144.78 0)
 			(effects
@@
 			)
 		)
-		(property "Footprint" "MountingHole:MountingHole_3mm"
+		(property "Footprint" "MountingHole:MountingHole_3.2mm_M3"
 			(at 331.47 139.7 0)
 			(effects
@@
 			)
 		)
-		(property "Footprint" "MountingHole:MountingHole_3mm"
+		(property "Footprint" "MountingHole:MountingHole_3.2mm_M3"
 			(at 326.39 144.78 0)
 			(effects
@@
 			)
 		)
-		(property "Footprint" "MountingHole:MountingHole_3mm"
+		(property "Footprint" "MountingHole:MountingHole_3.2mm_M3"
 			(at 326.39 139.7 0)
 			(effects
